File: Filters.kicad_sch (KiCad schematic)
At the start: 17 parts

Commit message: modular
Parts:
- removed C16, C17, C18: 100n, Capacitor_SMD:C_0603_1608Metric, symbol Device:C
- removed C19, C20, C21, C22, C23: 1n, Capacitor_SMD:C_0603_1608Metric, symbol Device:C
- removed JP1: VSel, Jumper:SolderJumper-3_P1.3mm_Bridged12_Pad1.0x1.5mm, symbol Jumper:Jumper_3_Bridged12
- removed R12, R13, R14, R15, R16, R17, R18, R19: 10k, Resistor_SMD:R_0603_1608Metric, symbol Device:R
Other:
- note removed: "10kHz Filters"
- note removed: "Input Voltage Filter"
- note removed: "Motor Temp Filter"
- note removed: "Sensor Voltage Selector"
- note removed: "Voltage Measure Filter"
