File: GigaMicroEPC.kicad_sch (KiCad schematic)
At the start: 29 parts, among them U1 STM32F405RGT6, Y1 X50328MSB2GI

Commit message: modular
Parts:
- removed C1, C2: 20p, Capacitor_SMD:C_0603_1608Metric, symbol Device:C
- removed C10, C12, C13, C6, C8: 100n, Capacitor_SMD:C_0603_1608Metric, symbol Device:C
- removed C11, C5, C7, C9: 10n, Capacitor_SMD:C_0603_1608Metric, symbol Device:C
- removed C3, C4: 1u, Capacitor_SMD:C_0603_1608Metric, symbol Device:C
- removed D1: L RUN, LED_SMD:LED_0603_1608Metric, symbol Device:LED
- removed D2: L FAULT, LED_SMD:LED_0603_1608Metric, symbol Device:LED
- removed R1, R2, R3, R4, R5: 10k, Resistor_SMD:R_0603_1608Metric, symbol Device:R
- removed TP1: NRST, TestPoint:TestPoint_Pad_1.0x1.0mm, symbol Connector:TestPoint
- removed U1: STM32F405RGT6, Package_QFP:LQFP-64_10x10mm_P0.5mm, symbol MCU_ST_STM32F4:STM32F405RGTx
- removed Y1: X50328MSB2GI, Crystal:Crystal_SMD_5032-2Pin_5.0x3.2mm, symbol Device:Crystal
- added J3: Main Connector, GigaVescLibs:X0802FVS-60AS-LPV01, symbol Connector_Generic:Conn_02x30_Odd_Even
Connections:
- net +3.3V: now also J3.57 (Pin_57), J3.59 (Pin_59)
- net CURR1 FILTERED: now also J3.13 (Pin_13)
- net CURR2 FILTERED: now also J3.23 (Pin_23)
- net CURR3 FILTERED: now also J3.33 (Pin_33)
- net GND: now also J3.5 (Pin_5), J3.6 (Pin_6), J3.60 (Pin_60), J3.7 (Pin_7)
- net H1: now also J3.17 (Pin_17)
- net H2: now also J3.27 (Pin_27)
- net H3: now also J3.37 (Pin_37)
- net I2C2 SCL/USART3 TX: now also J3.32 (Pin_32)
- net I2C2 SDA/USART3 RX: now also J3.34 (Pin_34)
- net IN V: now also J3.9 (Pin_9)
- net L1: now also J3.15 (Pin_15)
- net L2: now also J3.25 (Pin_25)
- net L3: now also J3.35 (Pin_35)
- net MOSTEMP1: now also J3.19 (Pin_19)
- net MOSTEMP2: now also J3.29 (Pin_29)
- net MOSTEMP3: now also J3.39 (Pin_39)
- net NRST: now also J3.12 (Pin_12)
- net POWER STAGE DISABLE: now also J3.41 (Pin_41)
- net POWER STAGE LOCKOUT: now also J3.43 (Pin_43)
- net SERVO: now also J3.55 (Pin_55)
- net SWCLK: now also J3.14 (Pin_14)
- net SWDIO: now also J3.16 (Pin_16)
- net USBD+: now also J3.18 (Pin_18)
- net USBD-: now also J3.20 (Pin_20)
- net VSENSE1: now also J3.11 (Pin_11)
- net VSENSE2: now also J3.21 (Pin_21)
- net VSENSE3: now also J3.31 (Pin_31)
- new net +12V: J3.1 (Pin_1), J3.3 (Pin_3)
- new net +5V: J3.2 (Pin_2), J3.4 (Pin_4)
- new net ESP IO9: J3.48 (Pin_48)
- new net ESP-IO0: J3.36 (Pin_36)
- new net ESP-IO1: J3.38 (Pin_38)
- new net ESP-IO10: J3.50 (Pin_50)
- new net ESP-IO18: J3.58 (Pin_58)
- new net ESP-IO19: J3.56 (Pin_56)
- new net ESP-IO5: J3.40 (Pin_40)
- new net ESP-IO6: J3.42 (Pin_42)
- new net ESP-IO7: J3.44 (Pin_44)
- new net ESP-IO8: J3.46 (Pin_46)
- new net ESPPROG RX: J3.54 (Pin_54)
- new net ESPPROG TX: J3.52 (Pin_52)
- new net HALL-VOLTAGE: J3.47 (Pin_47)
- new net HALL1 IN: J3.49 (Pin_49)
- new net HALL2 IN: J3.51 (Pin_51)
- new net HALL3 IN: J3.53 (Pin_53)
- new net IN-CANH: J3.10 (Pin_10)
- new net IN-CANL: J3.8 (Pin_8)
- new net SPI1-MISO-ADC2: J3.28 (Pin_28)
- new net SPI1-MOSI: J3.30 (Pin_30)
- new net SPI1-NSS: J3.24 (Pin_24)
- new net SPI1-SCK-ADC: J3.26 (Pin_26)
- new net TEMPMOTOR IN: J3.45 (Pin_45)
- no-connect marks 4 -> 0
Other:
- note removed: "CAN1 to ESP32"
- note removed: "Changed order vs DevKit"
- note removed: "Mutually exclusive with SPI1"
- note removed: "Same Header, either adc or spi"
- note removed: "USART3 or I2C2"
