File: IMU.kicad_sch (KiCad schematic)
At the start: 5 parts, among them U2 LSM6DS3TR-C

Commit message: modular
Parts:
- removed C14, C15: 100n, Capacitor_SMD:C_0603_1608Metric, symbol Device:C
- removed R10, R11: 4.7k, Resistor_SMD:R_0603_1608Metric, symbol Device:R
- removed U2: LSM6DS3TR-C, Package_LGA:Bosch_LGA-14_3x2.5mm_P0.5mm, symbol Sensor_Motion:BMI160
Connections:
- no-connect marks 6 -> 0
Other:
- note removed: "Accelerometer and Gyroscope"
- note removed: "Alternative: BMI270, BMI160 C2836813, C94021"
