File: Power.kicad_sch (KiCad schematic)
At the start: 20 parts, among them U4 TPS5430DDAR, U5 REF3033AIDBZR, U6 AMS1117-3.3

Commit message: modular
Parts:
- removed C28, C33, C34, C35: 22u, Capacitor_SMD:C_1206_3216Metric, symbol Device:C
- removed C29, C30: 1u, Capacitor_SMD:C_0603_1608Metric, symbol Device:C
- removed C31: 10n, Capacitor_SMD:C_0603_1608Metric, symbol Device:C
- removed C32, C36: 100uF 10V Tant, Capacitor_Tantalum_SMD:CP_EIA-6032-28_Kemet-C, symbol Device:C_Polarized_US
- removed D57: MM5Z5V6ST1G, Diode_SMD:D_SOD-523, symbol Diode:MM5Zxx
- removed D7: SS34, Diode_SMD:D_SMA, symbol Device:D_Schottky
- removed JP2: 5V-JMP, Jumper:SolderJumper-2_P1.3mm_Open_TrianglePad1.0x1.5mm, symbol Jumper:Jumper_2_Bridged
- removed JP3: 3.3V-JMP, Jumper:SolderJumper-2_P1.3mm_Open_TrianglePad1.0x1.5mm, symbol Jumper:Jumper_2_Bridged
- removed JP7: 12V-JMP, Jumper:SolderJumper-2_P1.3mm_Open_TrianglePad1.0x1.5mm, symbol Jumper:Jumper_2_Bridged
- removed L1: 15uH, Inductor_SMD:L_Bourns_SRP7028A_7.3x6.6mm, symbol Device:L_Iron
- removed R24: 10k, Resistor_SMD:R_0603_1608Metric, symbol Device:R
- removed R25: 3.3k, Resistor_SMD:R_0603_1608Metric, symbol Device:R
- removed U4: TPS5430DDAR, Package_SO:TI_SO-PowerPAD-8_ThermalVias, symbol Regulator_Switching:TPS5430DDA
- removed U5: REF3033AIDBZR, Package_TO_SOT_SMD:SOT-23, symbol Reference_Voltage:ISL21070CIH320Z-TK
- removed U6: AMS1117-3.3, Package_TO_SOT_SMD:SOT-223-3_TabPin2, symbol Regulator_Linear:AMS1117-3.3
Connections:
- no-connect marks 1 -> 0
Other:
- note removed: "12-16V -> 5V DCDC"
- note removed: "3.3V Voltage Reference"
- note removed: "5V -> 3.3V Regulator"
