File: Power.kicad_sch (KiCad schematic)
At the start: 0 parts

Commit message: initial
Parts:
- added C14, C15: 100n, Capacitor_SMD:C_0603_1608Metric, symbol Device:C
- added C23, C31, C41, C42: 22u, Capacitor_SMD:C_0603_1608Metric, symbol Device:C
- added C30: 47p, Capacitor_SMD:C_0603_1608Metric, symbol Device:C
- added C35, C36: 10u, Capacitor_SMD:C_0603_1608Metric, symbol Device:C
- added C37: 100p, Capacitor_SMD:C_0603_1608Metric, symbol Device:C
- added L3: 4.7u, Inductor_SMD:L_Sunlord_SWPA5040S, symbol Device:L
- added L4: 6.8u, Inductor_SMD:L_Sunlord_SWPA5040S, symbol Device:L
- added R10: 24k, Resistor_SMD:R_0603_1608Metric, symbol Device:R
- added R14: 68k, Resistor_SMD:R_0603_1608Metric, symbol Device:R
- added R16: 13k, Resistor_SMD:R_0603_1608Metric, symbol Device:R
- added R9: 75k, Resistor_SMD:R_0603_1608Metric, symbol Device:R
- added U3, U5: AP63356DV, GigaVescLibs:V-DFN3020-13_DIO, symbol GigaVescSymbols:AP63357DV
Connections:
- new net: C15.1, L4.1, U5.7 (NC), U5.9 (SW)
- new net: C37.1, R14.2, R16.1, U5.3 (FB)
- new net: C15.2, U5.6 (BST)
- new net: C30.1, R10.1, R9.2, U3.3 (FB)
- new net: C14.1, L3.1, U3.7 (NC), U3.9 (SW)
- new net: C14.2, U3.6 (BST)
- new net +12V: C35.1, C36.1, U3.1 (VIN), U3.2 (EN), U5.1 (VIN), U5.2 (EN)
- new net +3.3V: C23.1, C30.2, C31.1, L3.2, R9.1
- new net +5V: C37.2, C41.1, C42.1, L4.2, R14.1
- new net GND: C23.2, C31.2, C35.2, C36.2, C41.2, C42.2, R10.2, R16.2, U3.4 (COMP), U3.8 (GND), U5.4 (COMP), U5.8 (GND)
- no-connect marks 0 -> 2
Other:
- note added: "AP63356, 12V -> 3.3V, 450kHz fixed PWM (no light-load skipping) Vout = 0.8V ref * (1 + R9/R10) = 0.8 * (1 + 75k/24k) = 3.300V exact Feedforward cap C30: zero at 1/(2*pi*75k*47pF) = 45kHz (datasheet ref 91k/33pF = 53kHz, close enough, loop unaffected) Inductor L3 = 4.7uH (datasheet Table 1 value, do not change, internal comp) Ripple current: dIL = 3.3 * (1 - 3.3/12) / (4.7u * 450k) = 1.13A peak-pe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"
- note added: "AP63356, 12V -> 5V, 450kHz fixed PWM (no light-load skipping) Vout = 0.8V ref * (1 + R14/R16) = 0.8 * (1 + 68k/13k) = 4.985V (-0.3%) Feedforward cap C37: zero at 1/(2*pi*68k*100pF) = 23kHz (datasheet ref 157k/47pF = 22kHz, matched) Inductor L4 = 6.8uH (datasheet Table 1 value, do not change, internal comp) Ripple current: dIL = 5 * (1 - 5/12) / (6.8u * 450k) = 0.95A peak-peak inductor peak = load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"
- note added: "use inductors YSPI0520-4R7M and YSPI0520-6R8M"
