File: Supervisor.kicad_sch (KiCad schematic)
At the start: 4 parts, among them U16 ESP32-C3-WROOM-02-N4

Commit message: modular
Parts:
- removed C144: 100n, GigaVescLibs:C_0603_1608Metric_L, symbol Device:C
- removed R112, R113: 10k, Resistor_SMD:R_0603_1608Metric, symbol Device:R
- removed U16: ESP32-C3-WROOM-02-N4, GigaVescLibs:MODULE_ESP32-C3-WROOM-02-H4, symbol GigaVescSymbols:ESP32-C3-WROOM-02-N4
