File: CurrentSense.kicad_sch (KiCad schematic)
At the start: 16 parts, among them SW1 SW_SPDT, U2 THN10-7211UIR, U4 ZTP7193Y

Commit message: initial
Parts:
- removed C4, C8: 22u, Capacitor_SMD:C_1206_3216Metric, symbol Device:C
- removed C7: 100n, Capacitor_SMD:C_0402_1005Metric, symbol Device:C
- removed C9: 100uF 10V, Capacitor_Tantalum_SMD:CP_EIA-6032-28_Kemet-C, symbol Device:C_Polarized_US
- removed L1: 6.8u, Inductor_SMD:L_Chilisin_BMRB00050518-B, symbol Device:L_Iron
- removed NT1: NetTie_2, NetTie:NetTie-2_SMD_Pad2.0mm, symbol Device:NetTie_2
- removed R1: 20k, Resistor_SMD:R_0402_1005Metric, symbol Device:R
- removed R2: 2.7k, Resistor_SMD:R_0402_1005Metric, symbol Device:R
- removed R5: 100k, Resistor_SMD:R_0402_1005Metric, symbol Device:R
- removed R57, R58, R59: 348k, Resistor_SMD:R_0603_1608Metric, symbol Device:R
- removed R60: 18.7k, Resistor_SMD:R_0603_1608Metric, symbol Device:R
- removed SW1: SW_SPDT, symbol Switch:SW_SPDT
- removed U2: THN10-7211UIR, Converter_DCDC:Converter_DCDC_TRACO_THN10-xxxxUIR_THT, symbol Converter_DCDC:THN10-7211UIR
- removed U4: ZTP7193Y, Package_TO_SOT_SMD:SOT-23-6, symbol GigaVescSymbols:ZTP7193Y
- added C106, C136, C76: 2.2n, Capacitor_SMD:C_0603_1608Metric, symbol Device:C
- added C230, C240, C241: 100n, Capacitor_SMD:C_0402_1005Metric, symbol Device:C
- added C231: 1u, Capacitor_SMD:C_0603_1608Metric, symbol Device:C
- added C232, C233, C234: 10n, Capacitor_SMD:C_0603_1608Metric, symbol Device:C
- added R240, R241: 10k, Resistor_SMD:R_0402_1005Metric, symbol Device:R
- added R69, R82, R99: 150, Resistor_SMD:R_0603_1608Metric, symbol Device:R
- added TP37, TP38, TP39: CS, GigaVescLibs:TestPad-D1, symbol Connector:TestPoint
- added U30: INA4181A1IPWR, Package_SO:TSSOP-20_4.4x6.5mm_P0.65mm, symbol GigaDFN56:INA4181A1IPWR
- added U31: TLV2316, Package_SO:SOIC-8_3.9x4.9mm_P1.27mm, symbol Amplifier_Operational:LM2904
Connections:
- net GND: now also C106.2, C136.2, C230.2, C231.2, C240.2, C241.2, C76.2, R241.2, U30.16 (GND), U30.17 (IN+4), U30.18 (IN-4), U30.20 (REF4), U31.4 (V-)
- new net: U31.6 (-), U31.7
- new net +3.3V: C230.1, C231.1, C241.1, R240.1, U30.5 (VS), U31.8 (V+)
- new net 1V65_DIV: C240.1, R240.2, R241.1, U31.3 (+), U31.5 (+)
- new net 1V65_REF: U30.1 (REF1), U30.12 (REF3), U30.9 (REF2), U31.1, U31.2 (-)
- new net CS1_AMP: R69.1, U30.13 (OUT3)
- new net CS2_AMP: R82.1, U30.8 (OUT2)
- new net CS3_AMP: R99.1, U30.2 (OUT1)
- new net CURR1 FILTERED: C76.1, R69.2, TP37.1
- new net CURR2 FILTERED: C106.1, R82.2, TP38.1
- new net CURR3 FILTERED: C136.1, R99.2, TP39.1
- new net ISENSE1+: C232.1, U30.15 (IN+3)
- new net ISENSE1-: C232.2, U30.14 (IN-3)
- new net ISENSE2+: C233.1, U30.6 (IN+2)
- new net ISENSE2-: C233.2, U30.7 (IN-2)
- new net ISENSE3+: C234.1, U30.4 (IN+1)
- new net ISENSE3-: C234.2, U30.3 (IN-1)
Other:
- note added: "1.65 V reference buffer (INA REF pins need low impedance)"
- note added: "ADC RC: 150R + 2.2n at INA outputs -> control card"
- note added: "Differential input filter, place at U30 IN+/IN- pins (5 R source -> ~3 MHz)"
- note added: "Firmware: CURRENT_AMP_GAIN 20.0, CURRENT_SHUNT_RES (0.001/4)"
- note added: "Low-side phase current amplifier (INA4181A1, G = 20 V/V)"
- note added: "Place at U30 VS pin"
- note added: "Shunt: 4x 1 mOhm per phase, Kelvin-averaged -> 0.25 mOhm effective, +-324 A linear range"
- note added: "unused half: follower"
- note removed: "12-16V -> 5V DCDC"
- note removed: "Any DCDC brick 25.4x25.4 THN 10-7212WIR PQDE6W-Q110 RD5-110S12W"
- note removed: "Division up to 186V => 3.3V !!Those values have to be the same as on mosfet board!!"
- note removed: "For 100x220 enclosure"
- note removed: "Power supply for 200V applications"
