File: CurrentSense.kicad_sch (KiCad schematic)
At the start: 20 parts, among them U30 INA4181A1IPWR, U31 TLV2316

Commit message: gate resistors
Parts:
- added C242: 100n, Capacitor_SMD:C_0402_1005Metric, symbol Device:C
Connections:
- net +3.3V: no longer R240.1
- net GND: now also C242.2
- net 1V65_REF renamed +1.65REF
- net CURR1 FILTERED renamed CURR1-FILTERED
- net CURR2 FILTERED renamed CURR2-FILTERED
- net CURR3 FILTERED renamed CURR3-FILTERED
- new net +3.3REF: C242.1, R240.1
Other:
- moved on the sheet: C230, C231, C232, C233, C234, C240, C241, R240, R241, U31A, U31B, U31C
