File: GigaDFN56.kicad_pcb (KiCad board)
At the start: 4 copper layers, 100 x 60 mm, 207 parts, among them J1 MOTOR SENSORS, J2 CAN, J3 UART / I2C, J31 HX PZ1.0-2x10P WZ, J32 HX PZ1.0-2x10P WZ, J33 HX PZ1.0-2x10P WZ, J4 SPI / EXPANSION, J41 HX PZ1.0-2x10P WZ, J42 HX PZ1.0-2x10P WZ, J5 USB / SERVO, J6 Conn_02x03_Counter_Clockwise, Q1 ISC030N10NM6, Q10 ISC030N10NM6, Q11 ISC030N10NM6, Q12 ISC030N10NM6, Q13 ISC030N10NM6, Q14 ISC030N10NM6, Q15 ISC030N10NM6, Q16 ISC030N10NM6, Q17 ISC030N10NM6, Q18 ISC030N10NM6, Q19 ISC030N10NM6, Q2 ISC030N10NM6, Q20 ISC030N10NM6, Q21 ISC030N10NM6, Q22 ISC030N10NM6, Q23 ISC030N10NM6, Q24 ISC030N10NM6, Q3 ISC030N10NM6, Q4 ISC030N10NM6, Q5 ISC030N10NM6, Q6 ISC030N10NM6, Q7 ISC030N10NM6, Q8 ISC030N10NM6, Q9 ISC030N10NM6, U30 INA4181A1IPWR, U31 TLV2316, U6 2EDF7275K, U7 2EDF7275K, U8 2EDF7275K

Commit message: busbar
Parts:
- added H12: PhaseConnector, GigaDFN56:BusBar_5x2mm_L90, F.Cu at (155.5, 80.3)
- added H13: PhaseConnector, GigaDFN56:BusBar_5x2mm_L90, B.Cu at (155.5, 111.0)
