File: GigaDFN56.kicad_pcb (KiCad board)
At the start: 4 copper layers, 100 x 60 mm, 209 parts, among them J1 MOTOR SENSORS, J2 CAN, J3 UART / I2C, J31 HX PZ1.0-2x10P WZ, J32 HX PZ1.0-2x10P WZ, J33 HX PZ1.0-2x10P WZ, J4 SPI / EXPANSION, J41 HX PZ1.0-2x10P WZ, J42 HX PZ1.0-2x10P WZ, J5 USB / SERVO, J6 Conn_02x03_Counter_Clockwise, Q1 ISC030N10NM6, Q10 ISC030N10NM6, Q11 ISC030N10NM6, Q12 ISC030N10NM6, Q13 ISC030N10NM6, Q14 ISC030N10NM6, Q15 ISC030N10NM6, Q16 ISC030N10NM6, Q17 ISC030N10NM6, Q18 ISC030N10NM6, Q19 ISC030N10NM6, Q2 ISC030N10NM6, Q20 ISC030N10NM6, Q21 ISC030N10NM6, Q22 ISC030N10NM6, Q23 ISC030N10NM6, Q24 ISC030N10NM6, Q3 ISC030N10NM6, Q4 ISC030N10NM6, Q5 ISC030N10NM6, Q6 ISC030N10NM6, Q7 ISC030N10NM6, Q8 ISC030N10NM6, Q9 ISC030N10NM6, U30 INA4181A1IPWR, U31 TLV2316, U6 2EDF7275K, U7 2EDF7275K, U8 2EDF7275K

Commit message: gate resistors
Parts:
- added C242: 100n, Capacitor_SMD:C_0402_1005Metric, F.Cu at (128.5, 118.2)
- added R411: 4.7, GigaDFN56:R_0402_1005Metric_TightCrtYd, B.Cu at (120.0, 85.1)
- added R412: 4.7, GigaDFN56:R_0402_1005Metric_TightCrtYd, B.Cu at (126.4, 85.1)
- added R413: 4.7, GigaDFN56:R_0402_1005Metric_TightCrtYd, B.Cu at (132.8, 85.1)
- added R414: 4.7, GigaDFN56:R_0402_1005Metric_TightCrtYd, B.Cu at (113.6, 85.1)
- added R421: 4.7, GigaDFN56:R_0402_1005Metric_TightCrtYd, B.Cu at (163.5, 85.1)
- added R422: 4.7, GigaDFN56:R_0402_1005Metric_TightCrtYd, B.Cu at (157.1, 85.1)
- added R423: 4.7, GigaDFN56:R_0402_1005Metric_TightCrtYd, B.Cu at (150.7, 85.1)
- added R424: 4.7, GigaDFN56:R_0402_1005Metric_TightCrtYd, B.Cu at (144.3, 85.1)
- added R431: 4.7, GigaDFN56:R_0402_1005Metric_TightCrtYd, B.Cu at (175.0, 85.1)
- added R432: 4.7, GigaDFN56:R_0402_1005Metric_TightCrtYd, B.Cu at (187.8, 85.1)
- added R433: 4.7, GigaDFN56:R_0402_1005Metric_TightCrtYd, B.Cu at (181.4, 85.1)
- added R434: 4.7, GigaDFN56:R_0402_1005Metric_TightCrtYd, B.Cu at (194.2, 85.1)
- added R511: 4.7, GigaDFN56:R_0402_1005Metric_TightCrtYd, B.Cu at (120.0, 99.6)
- added R512: 4.7, GigaDFN56:R_0402_1005Metric_TightCrtYd, B.Cu at (126.4, 99.6)
- added R513: 4.7, GigaDFN56:R_0402_1005Metric_TightCrtYd, B.Cu at (132.8, 99.6)
- added R514: 4.7, GigaDFN56:R_0402_1005Metric_TightCrtYd, B.Cu at (113.6, 99.6)
- added R521: 4.7, GigaDFN56:R_0402_1005Metric_TightCrtYd, B.Cu at (150.7, 99.6)
- added R522: 4.7, GigaDFN56:R_0402_1005Metric_TightCrtYd, B.Cu at (157.1, 99.6)
- added R523: 4.7, GigaDFN56:R_0402_1005Metric_TightCrtYd, B.Cu at (163.5, 99.6)
- added R524: 4.7, GigaDFN56:R_0402_1005Metric_TightCrtYd, B.Cu at (144.3, 99.6)
- added R531: 4.7, GigaDFN56:R_0402_1005Metric_TightCrtYd, B.Cu at (181.4, 99.6)
- added R532: 4.7, GigaDFN56:R_0402_1005Metric_TightCrtYd, B.Cu at (187.8, 99.6)
- added R533: 4.7, GigaDFN56:R_0402_1005Metric_TightCrtYd, B.Cu at (194.2, 99.6)
- added R534: 4.7, GigaDFN56:R_0402_1005Metric_TightCrtYd, B.Cu at (175.0, 99.6)
- moved C234 21.3 mm to (154.0, 118.5), turned to -90 degrees
- moved C232 10.7 mm to (146.8, 111.5), turned to 180 degrees
- moved C233 8.94 mm to (149.8, 111.5), turned to 0 degrees
- moved R67 2.14 mm to (113.4, 102.2)
- moved R80 2.14 mm to (144.1, 102.2)
- moved R97 2.14 mm to (174.8, 102.2)
- moved C136 1.12 mm to (156.5, 120.8)
- moved R99 1.12 mm to (153.5, 120.8)
- moved TP39 1.12 mm to (155.0, 120.8)
- moved R82 0.54 mm to (154.0, 113.8)
- moved C128 0.40 mm to (173.3, 100.1)
- moved C68 0.40 mm to (111.9, 100.1)
- moved C98 0.40 mm to (142.6, 100.1)
- moved C230 0.30 mm to (153.5, 115.1)
- moved C231 0.30 mm to (153.9, 116.3)
Connections:
- net /CurrentSense/1V65_REF renamed /CurrentSense/+1.65REF
- net CURR1 FILTERED renamed CURR1-FILTERED
- net CURR2 FILTERED renamed CURR2-FILTERED
- net CURR3 FILTERED renamed CURR3-FILTERED
- net HALL1 IN renamed HALL1-IN
- net HALL2 IN renamed HALL2-IN
- net HALL3 IN renamed HALL3-IN
- net I2C2 SCL/USART3 TX renamed I2C2-SCL/USART3-TX
- net I2C2 SDA/USART3 RX renamed I2C2-SDA/USART3-RX
- net POWER STAGE DISABLE renamed POWER-STAGE-DISABLE
- net POWER STAGE LOCKOUT renamed POWER-STAGE-LOCKOUT
- net TEMPMOTOR IN renamed TEMPMOTOR-IN
- J31 pad 4: IN V -> +3.3REF
- J31 pad 8: GND -> IN-V
- Q1 pad 4: /DriverSocketPhase1/PH -> Net-(Q1-G)
- Q10 pad 4: /DriverSocketPhase1/PL -> Net-(Q10-G)
- Q11 pad 4: /DriverSocketPhase2/PL -> Net-(Q11-G)
- Q12 pad 4: /DriverSocketPhase3/PL -> Net-(Q12-G)
- Q13 pad 4: /DriverSocketPhase1/PH -> Net-(Q13-G)
- Q14 pad 4: /DriverSocketPhase1/PL -> Net-(Q14-G)
- Q15 pad 4: /DriverSocketPhase2/PH -> Net-(Q15-G)
- Q16 pad 4: /DriverSocketPhase2/PL -> Net-(Q16-G)
- Q17 pad 4: /DriverSocketPhase3/PH -> Net-(Q17-G)
- Q18 pad 4: /DriverSocketPhase3/PL -> Net-(Q18-G)
- Q19 pad 4: /DriverSocketPhase1/PH -> Net-(Q19-G)
- Q2 pad 4: /DriverSocketPhase2/PH -> Net-(Q2-G)
- Q20 pad 4: /DriverSocketPhase1/PL -> Net-(Q20-G)
- Q21 pad 4: /DriverSocketPhase2/PH -> Net-(Q21-G)
- Q22 pad 4: /DriverSocketPhase2/PL -> Net-(Q22-G)
- Q23 pad 4: /DriverSocketPhase3/PH -> Net-(Q23-G)
- Q24 pad 4: /DriverSocketPhase3/PL -> Net-(Q24-G)
- Q3 pad 4: /DriverSocketPhase3/PH -> Net-(Q3-G)
- Q4 pad 4: /DriverSocketPhase1/PH -> Net-(Q4-G)
- Q5 pad 4: /DriverSocketPhase2/PH -> Net-(Q5-G)
- Q6 pad 4: /DriverSocketPhase3/PH -> Net-(Q6-G)
- Q7 pad 4: /DriverSocketPhase1/PL -> Net-(Q7-G)
- Q8 pad 4: /DriverSocketPhase2/PL -> Net-(Q8-G)
- Q9 pad 4: /DriverSocketPhase3/PL -> Net-(Q9-G)
- R240 pad 1: +3.3V -> +3.3REF
- R59 pad 2: IN V -> IN-V
- R60 pad 1: IN V -> IN-V
Routing:
- net +BATT: track 53.2 -> 377.2 mm
- net IN V: track 63.8 -> 0.00 mm
- net IN-V: track 0.00 -> 63.7 mm
- net +3.3REF: track 0.00 -> 47.9 mm, vias 0 -> 2
- net GND: track 33.2 -> 37.6 mm, vias 346 -> 345
- net /DriverSocketPhase3/PL: track 27.8 -> 24.6 mm
- net /DriverSocketPhase2/PL: track 27.8 -> 24.6 mm
- net /DriverSocketPhase1/PL: track 27.8 -> 24.6 mm
- net /DriverSocketPhase2/PH: track 46.0 -> 43.4 mm
- net /DriverSocketPhase1/PH: track 46.0 -> 43.4 mm
- net /DriverSocketPhase3/PH: track 46.0 -> 43.4 mm
- net ISENSE2+: track 40.6 -> 42.6 mm
- net ISENSE2-: track 38.7 -> 40.7 mm
- net MOSTEMP2: track 50.0 -> 51.5 mm
- net MOSTEMP1: track 79.4 -> 80.9 mm
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