File: GigaDFN56.kicad_pcb (KiCad board)
At the start: 4 copper layers, 100 x 60 mm, 234 parts, among them J1 MOTOR SENSORS, J2 CAN, J3 UART / I2C, J31 HX PZ1.0-2x10P WZ, J32 HX PZ1.0-2x10P WZ, J33 HX PZ1.0-2x10P WZ, J4 SPI / EXPANSION, J41 HX PZ1.0-2x10P WZ, J42 HX PZ1.0-2x10P WZ, J5 USB / SERVO, J6 Conn_02x03_Counter_Clockwise, Q1 ISC030N10NM6, Q10 ISC030N10NM6, Q11 ISC030N10NM6, Q12 ISC030N10NM6, Q13 ISC030N10NM6, Q14 ISC030N10NM6, Q15 ISC030N10NM6, Q16 ISC030N10NM6, Q17 ISC030N10NM6, Q18 ISC030N10NM6, Q19 ISC030N10NM6, Q2 ISC030N10NM6, Q20 ISC030N10NM6, Q21 ISC030N10NM6, Q22 ISC030N10NM6, Q23 ISC030N10NM6, Q24 ISC030N10NM6, Q3 ISC030N10NM6, Q4 ISC030N10NM6, Q5 ISC030N10NM6, Q6 ISC030N10NM6, Q7 ISC030N10NM6, Q8 ISC030N10NM6, Q9 ISC030N10NM6, U30 INA4181A1IPWR, U31 TLV2316, U6 2EDF7275K, U7 2EDF7275K, U8 2EDF7275K

Commit message: clearance
Parts:
- NT1: footprint NetTie:NetTie-2_SMD_Pad2.0mm -> NetTie:NetTie-2_SMD_Pad0.5mm
- moved D9 13.6 mm to (181.7, 103.6), turned to 180 degrees
- moved D7 13.6 mm to (120.3, 103.6), turned to 180 degrees
- moved D8 13.6 mm to (151.0, 103.6), turned to 180 degrees
- moved R36 8.71 mm to (152.7, 105.5), turned to 180 degrees
- moved R33 8.71 mm to (122.0, 105.5), turned to 180 degrees
- moved R37 8.71 mm to (183.4, 105.5), turned to 180 degrees
- moved C6 2.78 mm to (131.1, 104.9), turned to 180 degrees
- moved C11 2.78 mm to (161.8, 104.9), turned to 180 degrees
- moved C13 2.78 mm to (192.5, 104.9), turned to 180 degrees
- moved C5 2.00 mm to (125.1, 99.7), turned to 0 degrees
- moved C10 2.00 mm to (155.8, 99.7), turned to 0 degrees
- moved C12 2.00 mm to (186.5, 99.7), turned to 0 degrees
- moved L11 1.97 mm to (132.1, 101.8)
- moved L12 1.97 mm to (162.8, 101.8)
- moved L13 1.97 mm to (193.5, 101.8)
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Routing:
- net +BATT: track 377.2 -> 701.2 mm
- net Net-(D9-K): track 13.6 -> 3.95 mm
- net Net-(D7-K): track 13.6 -> 3.95 mm
- net Net-(D8-K): track 13.6 -> 3.95 mm
- net +12V: track 157.8 -> 167.1 mm
- net +VSW: track 22.2 -> 25.2 mm
- net Net-(U6-OUTB): track 4.11 -> 6.16 mm
- net Net-(U8-OUTB): track 4.11 -> 6.16 mm
- net Net-(U7-OUTB): track 4.11 -> 6.16 mm
- net +3.3V: track 240.5 -> 242.3 mm
- net Net-(D8-A): track 1.99 -> 3.43 mm
- net Net-(D7-A): track 1.99 -> 3.43 mm
- net Net-(D9-A): track 1.99 -> 3.43 mm
- net /DriverSocketPhase1/P-GND: track 8.14 -> 6.84 mm
- net /DriverSocketPhase3/P-GND: track 8.14 -> 6.84 mm
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