File: DriverSocket.kicad_sch (KiCad schematic)
At the start: 51 parts, among them U10 STDRIVEG600, U11 ACS37030

Commit message: initial
Parts:
- removed C54, C55: 100p, Capacitor_SMD:C_0603_1608Metric, symbol Device:C
- removed C56, C57, C59, C60, C61, C62, C65, C66, C67: 220n 200V, Capacitor_SMD:C_1206_3216Metric, symbol Device:C
- removed C58, C63, C64: 4.7u 25v, Capacitor_SMD:C_0805_2012Metric, symbol Device:C
- removed C69, C70, C72, C73, C74, C75, C77, C78, C80, C81, C82, C83: 10u 100V, Capacitor_SMD:C_1210_3225Metric, symbol Device:C
- removed C71: 100n, Capacitor_SMD:C_0603_1608Metric, symbol Device:C
- removed C76: 2.2n, Capacitor_SMD:C_0603_1608Metric, symbol Device:C
- removed C79: 330u 200V, GigaVescLibs:CapacitorD18x32, symbol Device:C_Polarized
- removed D24: SS520F, Diode_SMD:D_SMA, symbol Device:D_Schottky
- removed D25: MM5Z5V6ST1G, Diode_SMD:D_SOD-523, symbol Diode:MM5Zxx
- removed D26: PESD5V0C1BSFYL, GigaVescLibs:DSN0603-2_0.6x0.3mm_P0.4mm, symbol Device:D_TVS
- removed JP4: PJ, GigaVescLibs:Jumper0.5, symbol Jumper:SolderJumper_2_Bridged
- removed R61, R62, R66: 2.2, Resistor_SMD:R_0603_1608Metric, symbol Device:R
- removed R63, R64: 10k, Resistor_SMD:R_0603_1608Metric, symbol Device:R
- removed R65: 4.7, Resistor_SMD:R_0603_1608Metric, symbol Device:R
- removed R68: 0.2m, Resistor_SMD:R_2512_6332Metric, symbol Device:R_US
- removed R69: 150, Resistor_SMD:R_0603_1608Metric, symbol Device:R
- removed R71: 348k, Resistor_SMD:R_0603_1608Metric, symbol Device:R
- removed U10: STDRIVEG600, Package_SO:SOIC-16_3.9x9.9mm_P1.27mm, symbol GigaVescSymbols:STDRIVEG600
- removed U11: ACS37030, GigaVescLibs:SOIC-6_3.9x4.9mm_P1.27mm, symbol GigaVescSymbols:ACS37030
- added C19, C20: 10u, Capacitor_SMD:C_0805_2012Metric, symbol Device:C
- added C26: 100n, Capacitor_SMD:C_0603_1608Metric, symbol Device:C
- added C5, C6: 4.7n, Capacitor_SMD:C_0603_1608Metric, symbol Device:C
- added D7: DSK320, Diode_SMD:D_SOD-123, symbol Device:D_Schottky
- added L11, L5: 470@100Mhz, Inductor_SMD:L_0603_1608Metric, symbol Device:L
- added R12, R30: 4.7, Resistor_SMD:R_0603_1608Metric, symbol Device:R
- added R17, R6: 10k, Resistor_SMD:R_0603_1608Metric, symbol Device:R
- added R33: 10, Resistor_SMD:R_0603_1608Metric, symbol Device:R
- added TP40: VS, GigaVescLibs:TestPad-D1, symbol Connector:TestPoint
- added TP46: VSN, GigaVescLibs:TestPad-D1, symbol Connector:TestPoint
- added U6: 2EDF7275K, GigaVescLibs:IC_2EDF7275KXUMA2, symbol GigaDFN56:2EDF7275K
- H7: footprint MountingHole:MountingHole_4.3mm_M4_Pad_Via -> MountingHole:MountingHole_4.3x6.2mm_M4_Pad; now left out of the parts list
Connections:
- net PHASE_OUT is gone; now on net VSW: H7.1
- net +3.3V: now also C26.2, U6.4 (SLDON), U6.7 (VDDI)
- net GND: now also C26.1, TP46.1, U6.1 (GNDI)
- net H: now also U6.2 (INA)
- net L: now also U6.3 (INB)
- net POWER STAGE LOCKOUT: now also U6.5 (DISABLE)
- net V SENSE: now also TP40.1
- net VSW: now also C19.2, C5.2, R6.2, U6.11 (GNDA)
- net at R70.2: now also R72.1
- new net: D7.2 (A), R33.2
- new net: L11.1, R30.1
- new net: R30.2, U6.9 (OUTB)
- new net: C19.1, D7.1 (K), U6.13 (VDDA)
- new net: L5.1, R12.1
- new net: R12.2, U6.12 (OUTA)
- new net +12V: C20.1, R33.1, U6.10 (VDDB)
- new net P-GND: C20.2, C6.2, R17.2, U6.8 (GNDB)
- new net PH: C5.1, L5.2, R6.1
- new net PL: C6.1, L11.2, R17.1
- no-connect marks 1 -> 0
Other:
- removed sheet FetPair
- added sheet FetPair3 (FetPair.kicad_sch)
- added sheet FetPair4 (FetPair.kicad_sch)
- sheet FetPair1 ports: added H, KS+, KS-, L, PHASE-GND; removed VGlH, VGlL, VGuH, VGuL, VSl
- sheet FetPair2 ports: added H, KS+, KS-, L, PHASE-GND; removed VGlH, VGlL, VGuH, VGuL, VSl
- note added: "Low-side shunt Kelvin sense: averaged across the 4 FET pairs, amplified on CurrentSense sheet"
- note added: "Or any shottky diode with 200V 0.5A <850mV forward voltage"
- note removed: "20uF total"
- note removed: "Boost to ~250A"
- note removed: "Boosted hall current sensor"
- note removed: "HF Loop Caps"
- note removed: "Intermediate Caps"
- note removed: "Or any shottky diode with 200V 5A <850mV forward voltage"
- note removed: "alternative: ACS725xLCTR-50AB ACS724LLCTR-50AB MT9223CT-50BR5"
- moved on the sheet: R70

Commit message: gate resistors
Connections:
- net POWER STAGE LOCKOUT renamed POWER-STAGE-LOCKOUT
- net V SENSE renamed V-SENSE
Changed lines of the file:
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@@
 		)
 	)
-	(global_label "POWER STAGE LOCKOUT"
-		(shape input)
+	(global_label "POWER-STAGE-LOCKOUT"
+		(shape output)
 		(at 45.72 73.66 180)
 		(fields_autoplaced yes)
@@
 		)
 	)
-	(hierarchical_label "V SENSE"
-		(shape input)
+	(hierarchical_label "V-SENSE"
+		(shape output)
 		(at 273.05 133.35 0)
 		(effects
@@
 	)
 	(hierarchical_label "MOS_TEMP"
-		(shape input)
+		(shape output)
 		(at 189.23 82.55 0)
 		(effects
@@
 			)
 		)
-		(pin "PHASE" input
+		(pin "PHASE" passive
 			(at 104.14 143.51 270)
 			(effects
@@
 			)
 		)
-		(pin "PHASE" input
+		(pin "PHASE" passive
 			(at 48.26 143.51 270)
 			(effects
@@
 			)
 		)
-		(pin "PHASE" input
+		(pin "PHASE" passive
 			(at 132.08 143.51 270)
 			(effects
@@
 			)
 		)
-		(pin "PHASE" input
+		(pin "PHASE" passive
 			(at 76.2 143.51 270)
 			(effects
