File: FetPair.kicad_sch (KiCad schematic)
At the start: 10 parts, among them Q1 EPC2304, Q2 EPC2304

Commit message: initial
Parts:
- removed D3, D4: RB751CM-40T2R, Diode_SMD:D_SOD-923, symbol Device:D_Schottky
- removed D5, D6: PESD5V0C1BSFYL, GigaVescLibs:DSN0603-2_0.6x0.3mm_P0.4mm, symbol Device:D_TVS
- removed Q1, Q2: EPC2304, GigaVescLibs:EPC-QFN3x5, symbol GigaVescSymbols:EPC2304
- removed R6, R8: 22, Resistor_SMD:R_0603_1608Metric, symbol Device:R
- removed R7, R9: 6.8, Resistor_SMD:R_0603_1608Metric, symbol Device:R
- added C2: 10u 100V, Capacitor_SMD:C_1210_3225Metric, symbol Device:C
- added C32: 100n, Capacitor_SMD:C_0805_2012Metric, symbol Device:C
- added Q1, Q7: ISC030N10NM6, Package_TO_SOT_SMD:TDSON-8-1, symbol Transistor_FET:BSC046N10NS3G
- added R111: 1m, Resistor_SMD:R_2512_6332Metric, symbol Device:R
- added R211, R311: 10, Resistor_SMD:R_0402_1005Metric, symbol Device:R
Connections:
- net +BATT: now also C2.1, C32.1, Q1.5 (D)
- net GND: now also C2.2, C32.2, R111.2, R311.2
- net PHASE: now also Q1.1 (S), Q1.2 (S), Q1.3 (S), Q7.5 (D)
- new net H: Q1.4 (G)
- new net KS+: R211.2
- new net KS-: R311.1
- new net L: Q7.4 (G)
- new net PHASE-GND: Q7.1 (S), Q7.2 (S), Q7.3 (S), R111.1, R211.1
Other:
- note added: "1 mOhm low-side shunt per FET pair, Kelvin-averaged (4x 10R per side)"
- note added: "10uF total"
- note removed: "Originally 15Ω and 1Ω but for 1 pair thats too much Per FET = 5V / 22Ω = 227mA Total = 3 * 227mA = 681mA"

Commit message: gate resistors
Parts:
- added R4**, R5**: 4.7, GigaDFN56:R_0402_1005Metric_TightCrtYd, symbol Device:R
Connections:
- net H: now also R4**.1; no longer Q1.4 (G)
- net L: now also R5**.1; no longer Q7.4 (G)
- new net: Q7.4 (G), R5**.2
- new net: Q1.4 (G), R4**.2

Commit message: clearance
Parts:
- renumbered R4** to R411, R5** to R511
