File: GigaDFN56.kicad_sch (KiCad schematic)
At the start: 22 parts, among them J31 HX PZ1.0-2x10P WZ, J32 HX PZ1.0-2x10P WZ, J33 HX PZ1.0-2x10P WZ, J41 HX PZ1.0-2x10P WZ, J42 HX PZ1.0-2x10P WZ

Commit message: busbar
Parts:
- added H12, H13: PhaseConnector, GigaDFN56:BusBar_5x2mm_L90, symbol Mechanical:MountingHole_Pad
Connections:
- net +BATT: now also H12.1
- net GND: now also H13.1

Commit message: gate resistors
Connections:
- net GND: no longer J31.8 (Pin_8)
- net CURR1 FILTERED renamed CURR1-FILTERED
- net CURR2 FILTERED renamed CURR2-FILTERED
- net CURR3 FILTERED renamed CURR3-FILTERED
- net HALL1 IN renamed HALL1-IN
- net HALL2 IN renamed HALL2-IN
- net HALL3 IN renamed HALL3-IN
- net I2C2 SCL/USART3 TX renamed I2C2-SCL/USART3-TX
- net I2C2 SDA/USART3 RX renamed I2C2-SDA/USART3-RX
- net IN V renamed IN-V
- net IN-V: now also J31.8 (Pin_8); no longer J31.4 (Pin_4)
- net POWER STAGE DISABLE renamed POWER-STAGE-DISABLE
- net POWER STAGE LOCKOUT renamed POWER-STAGE-LOCKOUT
- net TEMPMOTOR IN renamed TEMPMOTOR-IN
- new net +3.3REF: J31.4 (Pin_4)
Other:
- sheet DriverSocketPhase1 ports: added V-SENSE; removed V SENSE
- sheet DriverSocketPhase2 ports: added V-SENSE; removed V SENSE
- sheet DriverSocketPhase3 ports: added V-SENSE; removed V SENSE
- moved on the sheet: J31, J32

Commit message: clearance
Parts:
- NT1: footprint NetTie:NetTie-2_SMD_Pad2.0mm -> NetTie:NetTie-2_SMD_Pad0.5mm
Changed lines of the file:
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@@
 			)
 		)
-		(property "Footprint" "NetTie:NetTie-2_SMD_Pad2.0mm"
+		(property "Footprint" "NetTie:NetTie-2_SMD_Pad0.5mm"
 			(at 220.98 170.18 0)
 			(hide yes)
